File: pcb/thermal-station.sch (KiCad schematic (older format))
At the start: 38 parts, among them J1 Jack-DC, J2 Conn_01x03, J3 Conn_01x04_Male, Q1 AO3401A, SW1 RESET, SW2 SW_DIP_x02, SW3 FLASH, U1 ESP-12E, U10 KCSA02-105, U11 KCSA02-105, U12 DS18B20, U2 74HC595, U3 74HC595, U4 KCSA02-105, U5 KCSA02-105, U6 MH-Z19, U7 LM1117-3.3, U8 74HC595, U9 74HC595

Commit message: Redesign PCB
Parts:
- removed C2: CP, Capacitor_SMD:C_2816_7142Metric_Pad3.20x4.45mm_HandSolder, symbol Device:CP
- removed J1: Jack-DC, Connector_BarrelJack:BarrelJack_CUI_PJ-063AH_Horizontal, symbol Connector:Jack-DC
- removed J2: Conn_01x03, Connector_PinHeader_2.54mm:PinHeader_1x03_P2.54mm_Horizontal, symbol Connector_Generic:Conn_01x03
- removed J3: Conn_01x04_Male, Connector_PinHeader_2.54mm:PinHeader_1x04_P2.54mm_Vertical, symbol Connector:Conn_01x04_Male
- removed Q1: AO3401A, Package_TO_SOT_SMD:SOT-23, symbol Device:Q_PMOS_GSD
- removed R1, R9: R, Resistor_SMD:R_0805_2012Metric_Pad1.15x1.40mm_HandSolder, symbol Device:R
- removed RH1: AM2320, module:AM2320, symbol nosuz:AM2320
- removed RN1, RN2, RN3, RN4, RN5, RN6, RN7, RN8: R_Pack04, Resistor_SMD:R_Array_Convex_4x1206, symbol Device:R_Pack04
- removed RV1: R_POT, Potentiometer_THT:Potentiometer_Alps_RK09K_Single_Vertical, symbol Device:R_POT
- removed SW2: SW_DIP_x02, Button_Switch_THT:SW_DIP_SPSTx02_Piano_10.8x6.64mm_W7.62mm_P2.54mm, symbol Switch:SW_DIP_x02
- removed U10, U11, U4, U5: KCSA02-105, Display_7Segment:7SegmentLED_LTS6760_LTS6780, symbol Display_Character:KCSA02-105
- removed U12: DS18B20, Package_TO_SOT_THT:TO-92_Inline, symbol Sensor_Temperature:DS18B20
- removed U2, U3, U8, U9: 74HC595, Package_SO:SOIC-16W_7.5x10.3mm_P1.27mm, symbol 74xx:74HC595
- removed U6: MH-Z19, mh-z19:MH-Z19, symbol nrg3-cache:MH-Z19
- removed U7: LM1117-3.3, Package_TO_SOT_SMD:SOT-223-3_TabPin2, symbol Regulator_Linear:LM1117-3.3
- added C2, C3: 0.1uF, Capacitor_SMD:C_1206_3216Metric_Pad1.42x1.75mm_HandSolder, symbol Device:C
- C1: value C -> 0.1uF
- R1: renamed from R6; value R -> 10K
- R2: renamed from R5; value R -> 10K
- R3: renamed from R7; value R -> 10K
- R4: renamed from R8; value R -> 10K
- R5: renamed from R10; value R -> 10K
- SW1: footprint Button_Switch_SMD:SW_SPST_CK_RS282G05A3 -> Button_Switch_SMD:SW_SPST_TL3342
- SW2: renamed from SW3; footprint Button_Switch_SMD:SW_SPST_CK_RS282G05A3 -> Button_Switch_SMD:SW_SPST_TL3342
Connections:
- net +5V is gone; now on net ADC: C1.1
- net +3V3: now also C2.1, C3.1
- net Earth: now also C2.2, C3.2
- net RST: now reaches R2.1, SW1.2, U1.1 (REST)
- net GPIO0: now reaches R3.1, SW2.1, U1.12 (GPIO0)
- net RX renamed RXD
- net TX renamed TXD
- no-connect marks 17 -> 7
Other:
- moved on the sheet: R1, R2, R3, R4, R5, SW1, SW2, U1
